Commit message: Updated color for distal links

File: sr_description/hand/xacro/finger/distal/distal.urdf.xacro (robot description, xacro)
@@ -55,4 +55,7 @@
           </xacro:if>
         </geometry>
+        <material name="BiotacGreen">
+          <color rgba="0.31 0.85 0.42 1.0" />
+        </material>
       </visual>
       <collision>

File: sr_description/hand/xacro/thumb/thdistal.urdf.xacro (robot description, xacro)
@@ -141,6 +141,6 @@
             </xacro:if>
           </geometry>
-          <material name="shadow_thmiddle_material">
-            <color rgba="0.2 0.2 0.2 1.0" />
+          <material name="BiotacGreen">
+            <color rgba="0.31 0.85 0.42 1.0" />
           </material>
         </visual>
