Commit message: Further color updates

File: sr_description/hand/xacro/forearm/forearm_c.urdf.xacro (robot description, xacro)
@@ -30,7 +30,7 @@
     </material>
   </xacro:macro>
-  <xacro:macro name="grey" >
-    <material name="Grey">
-      <color rgba="0.90000 0.90000 0.90000 1.0" />
+  <xacro:macro name="black" >
+    <material name="Black">
+      <color rgba="0.0 0.0 0.0 1.0" />
     </material>
   </xacro:macro>
@@ -47,5 +47,5 @@
           <mesh filename="file://$(find sr_description)/meshes/components/forearm/forearm_${hand_version}.dae"/>
         </geometry>
-        <material name="Grey" />
+        <material name="Black" />
       </visual>
       <collision>

File: sr_description/hand/xacro/forearm/forearm_e.urdf.xacro (robot description, xacro)
@@ -30,7 +30,7 @@
     </material>
   </xacro:macro>
-  <xacro:macro name="light_grey" >
-    <material name="light_grey">
-      <color rgba="0.90000 0.90000 0.90000 1.0" />
+  <xacro:macro name="black" >
+    <material name="black">
+      <color rgba="0.0 0.0 0.0 1.0" />
     </material>
   </xacro:macro>
@@ -53,5 +53,5 @@
           <mesh filename="file://$(find sr_description)/meshes/components/forearm/forearm_${hand_version}.dae" scale="0.001 0.001 0.001" />
         </geometry>
-        <xacro:light_grey/>
+        <xacro:black/>
       </visual>
       <collision>

File: sr_description/hand/xacro/forearm/forearm_g.urdf.xacro (robot description, xacro)
@@ -44,5 +44,5 @@
           <mesh filename="file://$(find sr_description)/meshes/components/forearm/forearm_${hand_version}.dae" scale="1.0 1.0 1.0" />
         </geometry>
-        <material name="Grey" />
+        <material name="Black" />
       </visual>
       <collision>
